File: eagle/homecomputer-6502.sch (EAGLE design)
At the start: 61 parts, among them IC1 NE555, IC10 6522, IC11 6551, IC12 6581, IC2 74LS00N, IC3 74LS04N, IC4 74LS30N, IC5 74LS137N, IC6 6502, IC7 AT28C256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

Commit message: Add final schematics
Other:
- note added: "Final"
- note removed: "13"
Changed lines of the file:
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@@
 <plain>
 <text x="163.83" y="31.75" size="2.54" layer="94">Dirk Grappendorf</text>
-<text x="251.46" y="7.62" size="2.54" layer="94">13</text>
+<text x="251.46" y="7.62" size="2.54" layer="94">Final</text>
 <text x="163.83" y="27.94" size="2.54" layer="94">grappendorf.net</text>
 <text x="163.83" y="24.13" size="2.54" layer="94">CERN Open Hardware License 1.1</text>
@@
 <plain>
 <text x="163.83" y="31.75" size="2.54" layer="94">Dirk Grappendorf</text>
-<text x="251.46" y="7.62" size="2.54" layer="94">13</text>
+<text x="251.46" y="7.62" size="2.54" layer="94">Final</text>
 <text x="163.83" y="27.94" size="2.54" layer="94">grappendorf.net</text>
 <text x="163.83" y="24.13" size="2.54" layer="94">CERN Open Hardware License 1.1</text>
@@
 <plain>
 <text x="163.83" y="31.75" size="2.54" layer="94">Dirk Grappendorf</text>
-<text x="251.46" y="7.62" size="2.54" layer="94">13</text>
+<text x="251.46" y="7.62" size="2.54" layer="94">Final</text>
 <text x="163.83" y="27.94" size="2.54" layer="94">grappendorf.net</text>
 <text x="163.83" y="24.13" size="2.54" layer="94">CERN Open Hardware License 1.1</text>
@@
 <plain>
 <text x="163.83" y="31.75" size="2.54" layer="94">Dirk Grappendorf</text>
-<text x="251.46" y="7.62" size="2.54" layer="94">13</text>
+<text x="251.46" y="7.62" size="2.54" layer="94">Final</text>
 <text x="163.83" y="27.94" size="2.54" layer="94">grappendorf.net</text>
 <text x="163.83" y="24.13" size="2.54" layer="94">CERN Open Hardware License 1.1</text>
@@
 <plain>
 <text x="163.83" y="31.75" size="2.54" layer="94">Dirk Grappendorf</text>
-<text x="251.46" y="7.62" size="2.54" layer="94">13</text>
+<text x="251.46" y="7.62" size="2.54" layer="94">Final</text>
 <text x="163.83" y="27.94" size="2.54" layer="94">grappendorf.net</text>
 <text x="163.83" y="24.13" size="2.54" layer="94">CERN Open Hardware License 1.1</text>
